File: PCB Files/macro-microcontroller-2.kicad_pcb (KiCad board)
At the start: 2 copper layers, 96.5 x 35.6 mm, 48 parts, among them J1 USB_B_Micro, J2 SWD, J3 Barrel_Jack_MountingPin, J4 GPIO, M1 Motor_DC, SW1 Button, SW2 Button, SW3 Button, SW4 Reset, SW5 Controls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

Commit message: Update components
Parts:
- BZ1: value TMB12A24 -> HMB1206-03
Changed lines of the file:
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@@
 			)
 		)
+		(property "LCSC" "C84266"
+			(at 0 0 0)
+			(unlocked yes)
+			(layer "F.Fab")
+			(hide yes)
+			(effects
+				(font
+					(size 1 1)
+					(thickness 0.15)
+				)
+			)
+		)
 		(property ki_fp_filters "LED* LED_SMD:* LED_THT:*")
 		(sheetname "/")
@@
 			)
 		)
+		(property "LCSC" "C5156614"
+			(at 0 0 90)
+			(unlocked yes)
+			(layer "F.Fab")
+			(hide yes)
+			(effects
+				(font
+					(size 1 1)
+					(thickness 0.15)
+				)
+			)
+		)
 		(property ki_fp_filters "Connector*:*_1x??_*")
 		(sheetname "/")
@@
 			)
 		)
-		(property "Value" "TMB12A24"
+		(property "Value" "HMB1206-03"
 			(at 3.8 7.4 0)
 			(layer "F.Fab")
@@
 			)
 		)
-		(property "LCSC" "C96078"
+		(property "LCSC" "C96101"
 			(at 0 0 180)
 			(unlocked yes)

Commit message: Update PCB
Parts:
- added R9: 5kohm, Resistor_SMD:R_0402_1005Metric, F.Cu at (216.3, 99.6)
Connections:
- J2 pad 3: GND -> Net-(J2-~{RESET})
Routing:
- net Net-(J2-~{RESET}): track 0.00 -> 3.96 mm
- net +3V3: track 107.4 -> 108.9 mm
- net GND: track 42.4 -> 41.2 mm

Commit message: Update PCB
Parts:
- moved R2 1.78 mm to (162.3, 83.1)
- moved D1 1.78 mm to (172.7, 82.6)
- moved D2 1.78 mm to (165.0, 82.6)
- moved D3 1.78 mm to (157.2, 82.5)
- moved R4 1.78 mm to (170.1, 83.1)
- moved R5 1.78 mm to (177.7, 83.1)
- moved BZ1 0.89 mm to (189.5, 82.8)
- moved C5 0.41 mm to (207.6, 83.1)
Routing:
- net /LED3: track 50.7 -> 48.9 mm
- net /LED2: track 42.6 -> 40.8 mm
- net /LED1: track 34.8 -> 33.0 mm
- net GND: track 41.2 -> 39.9 mm
- net Net-(BZ1-+): track 22.5 -> 21.7 mm
- net /Motor_Pot: track 8.76 -> 8.25 mm
Other:
- board text added: "DC 5V"
- board text removed: "DC 9V"

Commit message: Update PCB
Parts:
- added REF**: Screw_Generic_2.0x3.0mm_SilkScreen, Symbol:Screw_Generic_2.0x3.0mm_SilkScreen, F.Cu at (215.5, 79.0)
- added REF**: ESD-Logo_6.6x6mm_SilkScreen, Symbol:ESD-Logo_6.6x6mm_SilkScreen, F.Cu at (181.7, 108.1)
- moved R5 0.13 mm to (177.8, 83.1)
Routing:
- net +3V3: track 108.9 -> 111.0 mm
- net GND: track 39.9 -> 41.7 mm, vias 6 -> 7
Other:
- board text added: "Electrostatic-sensitive device, handle with care!"
- board text added: "https://nicholas1023.github.io/macro-microcontroller-2/ 2026 Nicholas Lim. Open source."
- board text removed: "https://github.com/Nicholas1023/macro-microcontroller-2 2026 Nicholas Lim."
