File: PCB Files/macro-microcontroller-2.kicad_sch (KiCad schematic)
At the start: 47 parts, among them J1 USB_B_Micro, J2 SWD, J3 Barrel_Jack_MountingPin, J4 GPIO, M1 Motor_DC, SW1 Button, SW2 Button, SW3 Button, SW4 Reset, SW5 Controls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

Commit message: Update components
Parts:
- BZ1: value TMB12A24 -> HMB1206-03; LCSC C96078 -> C96101
Changed lines of the file:
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@@
 	(rectangle
 		(start 153.035 76.835)
-		(end 201.295 120.65)
+		(end 204.47 120.65)
 		(stroke
 			(width 0)
@@
 			)
 		)
-		(property "Value" "TMB12A24"
+		(property "Value" "HMB1206-03"
 			(at 190.5 104.1399 0)
 			(show_name no)
@@
 			)
 		)
-		(property "LCSC" "C96078"
+		(property "LCSC" "C96101"
 			(at 186.69 102.87 0)
 			(hide yes)

Commit message: Update PCB
Parts:
- added R9: 5kohm, Resistor_SMD:R_0402_1005Metric, symbol Device:R
Connections:
- net +3V3: now also R9.1
- net GND: no longer J2.3 (~{RESET})
- new net: J2.3 (~{RESET}), R9.2
Changed lines of the file:
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@@
 		)
 	)
+	(label "RUN"
+		(at 41.91 29.21 0)
+		(effects
+			(font
+				(size 1.27 1.27)
+			)
+			(justify left bottom)
+		)
+	)
 	(label "GPIO16"
 		(at 109.22 71.12 0)
@@
 	)
 	(symbol
-		(lib_id "power:GND")
-		(at 34.29 29.21 90)
-		(unit 1)
-		(body_style 1)
-		(exclude_from_sim no)
-		(in_bom yes)
-		(on_board yes)
-		(in_pos_files yes)
-		(dnp no)
-		(fields_autoplaced yes)
-		(property "Reference" "#PWR027"
-			(at 40.64 29.21 0)
-			(hide yes)
-			(show_name no)
-			(do_not_autoplace no)
-			(effects
-				(font
-					(size 1.27 1.27)
-				)
-			)
-		)
-		(property "Value" "GND"
-			(at 38.1 29.2099 90)
-			(show_name no)
-			(do_not_autoplace no)
-			(effects
-				(font
-					(size 1.27 1.27)
-				)
-				(justify right)
-			)
-		)
-		(property "Footprint" ""
-			(at 34.29 29.21 0)
-			(hide yes)
-			(show_name no)
-			(do_not_autoplace no)
-			(effects
-				(font
-					(size 1.27 1.27)
-				)
-			)
-		)
-		(property "Datasheet" ""
-			(at 34.29 29.21 0)
-			(hide yes)
-			(show_name no)
-			(do_not_autoplace no)
-			(effects
-				(font
-					(size 1.27 1.27)
-				)
-			)
-		)
-		(property "Description" "Power symbol creates a global label with name \"GND\" , ground"
-			(at 34.29 29.21 0)
-			(hide yes)
-			(show_name no)
-			(do_not_autoplace no)
-			(effects
-				(font
-					(size 1.27 1.27)
-				)
-			)
-		)
-		(pin "1"
-		)
-		(instances
-			(project "macro-microcontroller-2"
-				(path "/fde52755-4c02-4079-97f9-2f7863cc2631"
-					(reference "#PWR027")
-					(unit 1)
-				)
-			)
-		)
-	)
-	(symbol
 		(lib_id "MCU_RaspberryPi:RP2040")
 		(at 83.82 68.58 0)
@@
 					(unit 1)
 				)
+			)
+		)
+	)
+	(symbol
+		(lib_id "Device:R")
+		(at 38.1 29.21 270)
+		(unit 1)
+		(body_style 1)
+		(exclude_from_sim no)
+		(in_bom yes)
+		(on_board yes)
+		(in_pos_files yes)
+		(dnp no)
+		(fields_autoplaced yes)
+		(property "Reference" "R9"
+			(at 38.1 22.86 90)
+			(show_name no)
+			(do_not_autoplace no)
+			(effects
+				(font
+					(size 1.27 1.27)
+				)
+			)
+		)
+		(property "Value" "5kohm"
+			(at 38.1 25.4 90)
+			(show_name no)
+			(do_not_autoplace no)
+			(effects
+				(font
+					(size 1.27 1.27)
+				)
+			)
+		)
+		(property "Footprint" "Resistor_SMD:R_0402_1005Metric"
+			(at 38.1 27.432 90)
+			(hide yes)
+			(show_name no)
+			(do_not_autoplace no)
+			(effects
+				(font
+					(size 1.27 1.27)
+				)
+			)
+		)
+		(property "Datasheet" ""
+			(at 38.1 29.21 0)
+			(hide yes)
+			(show_name no)
+			(do_not_autoplace no)
+			(effects
+				(font
+					(size 1.27 1.27)
+				)
+			)
+		)
+		(property "Description" "Resistor"
+			(at 38.1 29.21 0)
+			(hide yes)
+			(show_name no)
+			(do_not_autoplace no)
+			(effects
+				(font
+					(size 1.27 1.27)
+				)
+			)
+		)
+		(property "LCSC" "C5948099"
+			(at 38.1 29.21 90)
+			(hide yes)
+			(show_name no)
+			(do_not_autoplace no)
+			(effects
+				(font
+					(size 1.27 1.27)
+				)
+			)
+		)
+		(property "KLC_S3.3" ""
+			(at 38.1 29.21 90)
+			(hide yes)
+			(show_name no)
+			(do_not_autoplace no)
+			(effects
+				(font
+					(size 1.27 1.27)
+				)
+			)
+		)
+		(property "KLC_S4.1" ""
+			(at 38.1 29.21 90)
+			(hide yes)
+			(show_name no)
+			(do_not_autoplace no)
+			(effects
+				(font
+					(size 1.27 1.27)
+				)
+			)
+		)
+		(property "KLC_S4.2_DVDD" ""
+			(at 38.1 29.21 90)
+			(hide yes)
+			(show_name no)
+			(do_not_autoplace no)
+			(effects
+				(font
+					(size 1.27 1.27)
+				)
+			)
+		)
+		(property "KLC_S4.2_VREG_VOUT" ""
+			(at 38.1 29.21 90)
+			(hide yes)
+			(show_name no)
+			(do_not_autoplace no)
+			(effects
+				(font
+					(size 1.27 1.27)
+				)
+			)
+		)
+		(pin "1"
+		)
+		(pin "2"
+		)
+		(instances
+			(project "macro-microcontroller-2"
+				(path "/fde52755-4c02-4079-97f9-2f7863cc2631"
+					(reference "R9")
+					(unit 1)
+				)

Commit message: Update PCB
Other:
- company: Designed by Nicholas Lim -> Designed by Nicholas Lim. Open source under the MIT License.
Changed lines of the file:
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@@
 	(title_block
 		(title "Macro Microcontroller 2")
-		(date "2026-06-19")
-		(rev "Rev 2")
-		(company "Designed by Nicholas Lim")
+		(date "2026-06-25")
+		(rev "2")
+		(company "Designed by Nicholas Lim. Open source under the MIT License.")
 		(comment 1 "Source: https://github.com/Nicholas1023/macro-microcontroller-2")
+		(comment 2 "Documentation: https://nicholas1023.github.io/macro-microcontroller-2")
 	)
 	(rectangle
