File: PCB Files/macro-microcontroller-2.kicad_sch (KiCad schematic)
At the start: 48 parts, among them J1 USB_B_Micro, J2 SWD, J3 Barrel_Jack_MountingPin, J4 GPIO, M1 Motor_DC, SW1 Button, SW2 Button, SW3 Button, SW4 Reset, SW5 Controls, SW6 Boot, U1 RP2040, U2 TLV71311PDBVR, U3 XC6206P332MR, U4 W25Q128JVP, U6 TPS76350, Y1 NX3225SA-12MHz

Commit message: Update schematics
Other:
- company: Designed by Nicholas Lim. Open source under the MIT License. -> Designed by Nicholas Lim. Open source under the CERN-OHL-P-2.0 License.
Changed lines of the file:
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@@
 		(date "2026-06-25")
 		(rev "2")
-		(company "Designed by Nicholas Lim. Open source under the MIT License.")
+		(company "Designed by Nicholas Lim. Open source under the CERN-OHL-P-2.0 License.")
 		(comment 1 "Source: https://github.com/Nicholas1023/macro-microcontroller-2")
 		(comment 2 "Documentation: https://nicholas1023.github.io/macro-microcontroller-2")

Commit message: Update schematics
Other:
- company: Designed by Nicholas Lim. Open source under the CERN-OHL-P-2.0 License. -> Designed by Nicholas Lim. Open source under the CERN-OHL-W-2.0 License.
Changed lines of the file:
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@@
 		(date "2026-06-25")
 		(rev "2")
-		(company "Designed by Nicholas Lim. Open source under the CERN-OHL-P-2.0 License.")
+		(company "Designed by Nicholas Lim. Open source under the CERN-OHL-W-2.0 License.")
 		(comment 1 "Source: https://github.com/Nicholas1023/macro-microcontroller-2")
 		(comment 2 "Documentation: https://nicholas1023.github.io/macro-microcontroller-2")
